Commit message: tmp

File: robot/abb_ws/src/abb_irb2400_support/urdf/irb2400_macro.xacro (robot description, xacro)
@@ -294,5 +294,5 @@
     <!-- end of joint list -->
     <joint name="kinect_joint" type="fixed">
-        <origin xyz="1.0 0.0 1.35" rpy="0.0 0.0 3.14159265359"/>
+        <origin xyz="1.5 0.0 1.35" rpy="0.0 0.0 3.14159265359"/>
         <parent link="world"/>
         <child link="kinect_link"/>
